File: schematics/libredaq-eagle-boards/LDAQ-MOD-ADC8/LDAQ-MOD-ADC8.brd (EAGLE design)
At the start: 17 parts, among them CON1 BOARD, IC1 24C01ASN, J1 ADC[0-7], SW1 SW_DIP-4, U1 AD7606

Commit message: update adc8 board
Parts:
- removed U1: AD7606, libredaq-comps:LQFP-ST-64-2
- added IC2: AD7606BSTZ, SamacSys_Parts:QFP50P1200X1200X160-64N
- C1, C3, C4, C7: device SparkFun-Capacitors:0603-CAP -> LMK105BJ225KV-F:CAPC1005X55N
- C2: device SparkFun-Capacitors:EIA3216 -> TAJB226M010RNJ:CAPPM3528X210N
- C5, C6: device SparkFun-Capacitors:0603-CAP -> 885012105010:CAPC1005X55N
- IC1: value 24C01ASN -> M24C02-FMN6TP; device libredaq-comps:SO-08 -> SamacSys_Parts:SOIC127P600X175-8N
- moved C7 3.56 mm to (28.0, 40.4)
- moved C4 0.28 mm to (29.3, 40.4)
- moved IC1 0.13 mm to (19.1, 15.8), turned to 90 degrees
- moved C2 0.05 mm to (36.6, 36.8), turned to 90 degrees
Connections:
- removed net N$17: R4.2, SW1.B3, U1.4
- removed net N$18: R4.1, SW1.B4, U1.5
- removed net N$33: C4.1, U1.39
- removed net N$34: C7.1, U1.36
- removed net N$36: J1.9, U1.49
- removed net N$37: J1.8, U1.51
- removed net N$38: J1.7, U1.53
- removed net N$39: J1.6, U1.55
- removed net N$40: J1.5, U1.57
- removed net N$41: J1.4, U1.59
- removed net N$42: J1.3, U1.61
- removed net N$43: J1.2, U1.63
- removed net N$44: C1.2, U1.44, U1.45
- removed net N$5: R4.3, SW1.B2, U1.3
- new net N$1: C1.2, IC2.44, IC2.45
- new net N$2: C4.1, IC2.36
- new net OS0: IC2.3, R4.3, SW1.B2
- new net OS1: IC2.4, R4.2, SW1.B3
- new net OS2: IC2.5, R4.1, SW1.B4
- new net RANGE: IC2.8, R4.4, SW1.B1
- new net V1: IC2.49, J1.9
- new net V2: IC2.51, J1.8
- new net V3: IC2.53, J1.7
- new net V4: IC2.55, J1.6
- new net V5: IC2.57, J1.5
- new net V6: IC2.59, J1.4
- new net V7: IC2.61, J1.3
- new net V8: IC2.63, J1.2
- net !DAQ_RD: now also IC2.12, IC2.13; no longer U1.12, U1.13
- net 3.3V: now also IC2.23, IC2.33, IC2.34, IC2.6, IC2.7; no longer U1.23, U1.33, U1.34, U1.6, U1.7
- net ADC_VCC: now also C2.1, IC2.1, IC2.37, IC2.38, IC2.48; no longer C2.A, U1.1, U1.37, U1.38, U1.48
- net AGND: now also C2.2, IC2.2, IC2.26, IC2.35, IC2.40, IC2.41, IC2.43, IC2.46, IC2.47, IC2.50, IC2.52, IC2.54, IC2.56, IC2.58, IC2.60, IC2.62, IC2.64; no longer C2.C, U1.2, U1.26, U1.35, U1.40, U1.41, U1.43, U1.46, U1.47, U1.50, U1.52, U1.54, U1.56, U1.58, U1.60, U1.62, U1.64
- net DAQ_1STDATA: now also IC2.15; no longer U1.15
- net DAQ_BUSY: now also IC2.14; no longer U1.14
- net DAQ_CONVST: now also IC2.10, IC2.9; no longer U1.10, U1.9
- net DAQ_RESET: now also IC2.11; no longer U1.11
- net DATA0: now also IC2.16; no longer U1.16
- net DATA1: now also IC2.17; no longer U1.17
- net DATA2: now also IC2.18; no longer U1.18
- net DATA3: now also IC2.19; no longer U1.19
- net DATA4: now also IC2.20; no longer U1.20
- net DATA5: now also IC2.21; no longer U1.21
- net DATA6: now also IC2.22; no longer U1.22
- net DATA7: now also IC2.24; no longer U1.24
- net N$3: now also C7.1, IC2.39; no longer R4.4, SW1.B1, U1.8
- net N$35: now also IC2.42; no longer U1.42
Routing:
- net OS0: track 0.00 -> 38.8 mm, vias 0 -> 2
- net RANGE: track 0.00 -> 37.1 mm, vias 0 -> 2
- net N$5: track 36.3 -> 0.00 mm, vias 2 -> 0
- net OS1: track 0.00 -> 35.7 mm, vias 0 -> 2
- net OS2: track 0.00 -> 34.9 mm, vias 0 -> 2
- net N$18: track 33.6 -> 0.00 mm, vias 2 -> 0
- net N$17: track 33.0 -> 0.00 mm, vias 2 -> 0
- net N$3: track 36.2 -> 4.50 mm, vias 2 -> 0
- net N$36: track 20.8 -> 0.00 mm
- net V1: track 0.00 -> 20.6 mm
- net N$37: track 19.7 -> 0.00 mm
- net N$38: track 18.7 -> 0.00 mm
- net V2: track 0.00 -> 18.4 mm
- net N$43: track 18.1 -> 0.00 mm
- net N$39: track 17.6 -> 0.00 mm
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
Commit message: done with adc8 board
Parts:
- CON1: device libredaq-comps:PCI-E_64_EDGE_63X50_PADS-ONLY -> libredaq-comps:PCI-E_64_EDGE_63X50
Routing:
- net 3.3V_EEP: track 15.8 -> 16.3 mm
Other:
- board outline added: 63 x 49.5 mm
Changed lines of the file:
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@@
 </element>
 <element name="SJ2" library="SparkFun-Passives" package="PAD-JUMPER-2-NC_BY_PASTE_YES_SILK" value="JUMPER-PAD-2-NC_BY_PASTE" x="40.02" y="38.94" smashed="yes" rot="R180"/>
-<element name="CON1" library="libredaq-comps" package="PCI-E_64_EDGE_63X50_PADS-ONLY" value="BOARD" x="25" y="0" smashed="yes"/>
+<element name="CON1" library="libredaq-comps" package="PCI-E_64_EDGE_63X50" value="BOARD" x="25" y="0" smashed="yes"/>
 <element name="LOGO1" library="libredaq-comps" package="LIBREDAQ_LOGO" value="LIBREDAQ_LOGO_MINILOGO_GENERIC" x="42" y="34" smashed="yes"/>
 <element name="R4" library="SparkFun-Resistors" package="0603-ARV" value="100k" x="51" y="32" smashed="yes">
@@
 <attribute name="MOUSER_PRICE-STOCK" value="https://www.mouser.co.uk/ProductDetail/STMicroelectronics/M24C02-FMN6TP?qs=WHlX%252B%252B9%2FRwCvVyrf2ztAog%3D%3D" x="19.079" y="15.844" size="1.778" layer="27" rot="R90" display="off"/>
 <attribute name="NAME" x="15.079" y="13.844" size="1.27" layer="25" rot="R90" align="center"/>
-<attribute name="VALUE" x="12.079" y="11.844" size="1.27" layer="27" rot="R90" align="center"/>
 </element>
 <element name="IC2" library="SamacSys_Parts" package="QFP50P1200X1200X160-64N" value="AD7606BSTZ" x="26.709" y="30.208" smashed="yes" rot="R90">
@@
 <wire x1="17.45" y1="14.55" x2="15.5" y2="16.5" width="0.254" layer="16"/>
 <contactref element="CON1" pad="A5"/>
-<wire x1="17.45" y1="4.25" x2="17.45" y2="14.55" width="0.254" layer="16"/>
+<wire x1="17.45" y1="3.75" x2="17.45" y2="14.55" width="0.254" layer="16"/>
 <contactref element="IC1" pad="8"/>
 <wire x1="17.174" y1="18.556" x2="15.5" y2="16.882" width="0.254" layer="1"/>
